File: usb-C adapter.kicad_sch (KiCad schematic)
At the start: 12 parts

Commit message: feat(no-headphone-usb-c-adapter-shrunk-down): NA
Parts:
- gave numbers to parts that had none: 1
- renumbered R3 to R33
Connections:
- net at U1.2 (VIN): now also C1.2, pchannel.3 (S)
Changed lines of the file:
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@@
   (symbol (lib_id "usb-c:IP2721") (at 147.32 67.31 90) (unit 1)
     (in_bom yes) (on_board yes) (fields_autoplaced)
-    (property "Reference" "U?" (id 0) (at 160.02 66.0399 90)
+    (property "Reference" "U1" (id 0) (at 160.02 66.0399 90)
       (effects (font (size 1.27 1.27)) (justify right))
     )
@@
   (symbol (lib_id "Device:R") (at 107.95 31.75 0) (unit 1)
     (in_bom yes) (on_board yes)
-    (property "Reference" "R3" (id 0) (at 105.41 31.75 90))
+    (property "Reference" "R33" (id 0) (at 105.41 31.75 90))
     (property "Value" "5.1kOhm" (id 1) (at 107.95 31.75 90)
       (effects (font (size 0.85 0.85)))
@@
       (reference "R3") (unit 1) (value "5.1kOhm") (footprint "")
     )
-    (path "/9b62e7e6-bf07-4ae3-bb33-5f179935ea9d"
-      (reference "R3") (unit 1) (value "5.1kOhm") (footprint "")
-    )
     (path "/00c27ddd-2126-493f-a3e8-14b303ff8a20"
       (reference "R4") (unit 1) (value "15kOhm") (footprint "")
@@
       (reference "R4") (unit 1) (value "15kOhm") (footprint "")
     )
+    (path "/9b62e7e6-bf07-4ae3-bb33-5f179935ea9d"
+      (reference "R33") (unit 1) (value "5.1kOhm") (footprint "")
+    )
     (path "/238ea9d6-a9e4-4569-a775-7a6321883506"
-      (reference "U?") (unit 1) (value "IP2721") (footprint "")
+      (reference "U1") (unit 1) (value "IP2721") (footprint "")
     )
     (path "/cebee702-107b-4d2c-820b-a13171e07761"
